Commit message: Fix URDF: add xacro namespace, gazebo materials, and sensor plugins

File: urdf/s500_quadcopter.urdf (robot description, URDF)
Before this commit: robot s500_quadcopter, 14 links, 13 joints
Joints:
- joint arm_fl_joint: origin xyz=0 0 0 rpy=0 0 0 -> xyz=0.0 0.0 0.0 rpy=0 0 0
- joint arm_fr_joint: origin xyz=0 0 0 rpy=0 0 0 -> xyz=0.0 0.0 0.0 rpy=0 0 0
- joint arm_rl_joint: origin xyz=0 0 0 rpy=0 0 0 -> xyz=0.0 0.0 0.0 rpy=0 0 0
- joint arm_rr_joint: origin xyz=0 0 0 rpy=0 0 0 -> xyz=0.0 0.0 0.0 rpy=0 0 0
- joint motor_fl_joint: limit (none) -> effort=10 velocity=100
- joint motor_fr_joint: limit (none) -> effort=10 velocity=100
- joint motor_rl_joint: limit (none) -> effort=10 velocity=100
- joint motor_rr_joint: limit (none) -> effort=10 velocity=100

Commit message: Update 5/6/26

File: urdf/s500_quadcopter.urdf (robot description, URDF)
Before this commit: robot s500_quadcopter, 14 links, 13 joints
Links:
- removed link motor_fl
- removed link motor_fr
- removed link motor_rl
- removed link motor_rr
- added link landing_leg_left, mass 0.001; collision cylinder length=0.240 radius=0.006; visual cylinder length=0.012 radius=0.0068
- added link landing_leg_right, mass 0.001; collision cylinder length=0.240 radius=0.006; visual cylinder length=0.012 radius=0.0068
- link arm_fl: mass 0.08 -> 0.001; geometry collision box size=0.25 0.015 0.015; visual box size=0.25 0.015 0.015
- link arm_fr: mass 0.08 -> 0.001; geometry collision box size=0.25 0.015 0.015; visual box size=0.25 0.015 0.015
- link arm_rl: mass 0.08 -> 0.001; geometry collision box size=0.25 0.015 0.015; visual box size=0.25 0.015 0.015
- link arm_rr: mass 0.08 -> 0.001; geometry collision box size=0.25 0.015 0.015; visual box size=0.25 0.015 0.015
- link base_link: mass 0.45 -> 1.1; geometry collision box size=0.165 0.165 0.025; visual box size=0.055 0.055 0.028
- link battery: mass 0.38 -> 0.001; geometry collision box size=0.135 0.042 0.025; visual box size=0.135 0.042 0.025
- link prop_fl: mass 0.05 -> 0.001; geometry collision cylinder length=0.008 radius=0.127; visual cylinder length=0.008 radius=0.127
- link prop_fr: mass 0.05 -> 0.001; geometry collision cylinder length=0.008 radius=0.127; visual cylinder length=0.008 radius=0.127
- link prop_rl: mass 0.05 -> 0.001; geometry collision cylinder length=0.008 radius=0.127; visual cylinder length=0.008 radius=0.127
- link prop_rr: mass 0.05 -> 0.001; geometry collision cylinder length=0.008 radius=0.127; visual cylinder length=0.008 radius=0.127
Joints:
- added joint landing_leg_left_joint: type fixed, parent base_link, child landing_leg_left, origin xyz=0 -0.090 -0.095 rpy=0 0 0
- added joint landing_leg_right_joint: type fixed, parent base_link, child landing_leg_right, origin xyz=0 0.090 -0.095 rpy=0 0 0
- joint arm_fl_joint: origin xyz=0.0 0.0 0.0 rpy=0 0 0 -> xyz=0 0 0 rpy=0 0 -0.7854
- joint arm_fr_joint: origin xyz=0.0 0.0 0.0 rpy=0 0 0 -> xyz=0 0 0 rpy=0 0 0.7854
- joint arm_rl_joint: origin xyz=0.0 0.0 0.0 rpy=0 0 0 -> xyz=0 0 0 rpy=0 0 -0.7854
- joint arm_rr_joint: origin xyz=0.0 0.0 0.0 rpy=0 0 0 -> xyz=0 0 0 rpy=0 0 0.7854
- joint battery_joint: origin xyz=0 0 0 rpy=0 0 0 -> xyz=0 0 -0.024 rpy=0 0 0
- joint motor_fl_joint: limit effort=10 velocity=100 -> effort=10 velocity=670; origin xyz=0.25 0 0 rpy=0 0 0 -> xyz=0.25 0 0.015 rpy=0 0 0
- joint motor_fr_joint: limit effort=10 velocity=100 -> effort=10 velocity=670; origin xyz=0.25 0 0 rpy=0 0 0 -> xyz=0.25 0 0.015 rpy=0 0 0
- joint motor_rl_joint: limit effort=10 velocity=100 -> effort=10 velocity=670; origin xyz=-0.25 0 0 rpy=0 0 0 -> xyz=-0.25 0 0.015 rpy=0 0 0
- joint motor_rr_joint: limit effort=10 velocity=100 -> effort=10 velocity=670; origin xyz=-0.25 0 0 rpy=0 0 0 -> xyz=-0.25 0 0.015 rpy=0 0 0
- joint prop_fl_joint: origin xyz=0 0 0.02 rpy=0 0 0 -> xyz=0 0 0.020 rpy=0 0 0
- joint prop_fr_joint: origin xyz=0 0 0.02 rpy=0 0 0 -> xyz=0 0 0.020 rpy=0 0 0
- joint prop_rl_joint: origin xyz=0 0 0.02 rpy=0 0 0 -> xyz=0 0 0.020 rpy=0 0 0
- joint prop_rr_joint: origin xyz=0 0 0.02 rpy=0 0 0 -> xyz=0 0 0.020 rpy=0 0 0
